File: ISysProgrammingTrainerTypeA/ISysProgrammingTrainerTypeA.kicad_pcb (KiCad board)
At the start: 2 copper layers, 95 x 72 mm, 20 parts, among them J1 Conn_01x15_Socket, J2 Conn_01x15_Socket, J3 Conn_01x05_Socket, J4 Conn_01x05_Socket, SW1 SW_Push, SW2 SW_Push, U1 74HC595, U2 ULN2803A

Commit message: シルク印刷にリポジトリのリンクを追加
Other:
- board text added: "https://github.com/I-Sys-UF/Trainer/"
Changed lines of the file:
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@@
     (effects (font (size 1.5 1.5) (thickness 0.2)) (justify left))
+  )
+  (gr_text "https://github.com/I-Sys-UF/Trainer/" (at 190.5 134.62) (layer "B.SilkS")
+    (effects (font (size 1.5 1.5) (thickness 0.2)) (justify left mirror))
   )
   (gr_text "I.Sys Programming Trainer Type-A v1" (at 147.32 134.62) (layer "F.SilkS")

Commit message: シルク印刷を追加
`Arduino Nano` の刻印を追加
Other:
- board text added: "Arduino Nano"
Changed lines of the file:
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@@
     (effects (font (size 1.5 1.5) (thickness 0.2)) (justify left))
+  )
+  (gr_text "Arduino Nano" (at 116.84 83.058) (layer "F.SilkS")
+    (effects (font (size 1 1) (thickness 0.15)))
   )
   (dimension (type aligned) (layer "Dwgs.User")
